Commit message: Update ridgeback_dual_ur5_description.urdf.xacro

File: betago_description/urdf/betago/ridgeback_dual_ur5_description.urdf.xacro (robot description, xacro)
@@ -1,13 +1,22 @@
 <?xml version="1.0"?>
 <robot xmlns:xacro="http://ros.org/wiki/xacro">
+<!--////////////////////////////////////Aluminum profile frame/////////////////////////////////////////-->
+  <xacro:include filename="$(find betago_description)/urdf/ridgeback/frame_link.urdf" />
+  <joint name="mid_mount_plus" type="fixed">
+    <parent link="mid_mount" />
+    <child link="basef_link" />
+    <origin xyz="0.21 0.0 0.0" rpy="0 0 0" />
+  </joint>
   <joint name="left_arm_mount_joint" type="fixed">
-    <parent link="mid_mount" />
+    <parent link="connect_Link" />
     <child link="left_ur_arm_base_link" />
-    <origin xyz="$(optenv RIDGEBACK_LEFT_UR_XYZ 0.21 0.20 0.0)" rpy="$(optenv RIDGEBACK_LEFT_UR_RPY 0 0 0)"/>
+    <origin xyz="0.0 0.0 0.0" rpy="1.5708 0 0" />
+  <!--<origin xyz="$(optenv RIDGEBACK_LEFT_UR_XYZ 0.21 0.20 0.0)" rpy="$(optenv RIDGEBACK_LEFT_UR_RPY 0 0 0)"/> -->
   </joint>
   <joint name="right_arm_mount_joint" type="fixed">
-    <parent link="mid_mount" />
+    <parent link="connect2_Link" />
     <child link="right_ur_arm_base_link" />
-    <origin xyz="$(optenv RIDGEBACK_RIGHT_UR_XYZ 0.21 -0.20 0.0)" rpy="$(optenv RIDGEBACK_RIGHT_UR_RPY 0 0 0)"/>
+    <origin xyz="0.0 0.0 0.0" rpy="1.5708 3.1416 0" />
+  <!-- <origin xyz="$(optenv RIDGEBACK_RIGHT_UR_XYZ 0.21 -0.20 0.0)" rpy="$(optenv RIDGEBACK_RIGHT_UR_RPY 0 0 0)"/> -->
   </joint>
   <xacro:include filename="$(find betago_description)/urdf/ur5/ur5.urdf.xacro" />
