Commit message: betago rtabmap demo

File: betago_description/urdf/betago/ridgeback_urdf_extras.xacro (robot description, xacro)
@@ -2,4 +2,4 @@
 <robot name="betago" xmlns:xacro="http://ros.org/wiki/xacro">
     <xacro:include filename="$(find betago_description)/urdf/betago/ridgeback_dual_ur5_description.urdf.xacro" />
-    <xacro:include filename="$(find betago_description)/urdf/allegro_hand/dual_allegro_hand.xacro" />
+<!--    <xacro:include filename="$(find betago_description)/urdf/allegro_hand/dual_allegro_hand.xacro" /> -->
 </robot>

File: betago_description/urdf/ridgeback/ridgeback.urdf.xacro (robot description, xacro)
@@ -1,5 +1,6 @@
 <?xml version="1.0"?>
 <robot name="ridgeback" xmlns:xacro="http://ros.org/wiki/xacro">
-  <xacro:property name="PI" value="3.1415926535897931" />
+    <xacro:property name="PI" value="3.1415926535897931" />
+    <xacro:property name="M_PI" value="3.1415926535897931" />
   <xacro:property name="wheel_radius" value="0.0759" />
   <xacro:property name="wheel_width" value="0.0790" />
@@ -272,3 +273,13 @@
   <!-- Optional custom includes. -->
   <xacro:include filename="$(optenv RIDGEBACK_URDF_EXTRAS empty.urdf)" />
+  <!-- sensors -->
+  <xacro:include filename="$(find betago_description)/urdf/sensors/kinect.urdf.xacro" />
+  <sensor_kinect  parent="base_link"/>
+<!--  <xacro:include filename="$(find betago_description)/urdf/sensors/kinect_gazebo.xacro" />-->
+<!--  <xacro:kinect_camera prefix="kinect" />-->
+<!--  <joint name="camera_joint" type="fixed">-->
+<!--    <origin xyz="-0.087 0.0 1.1" rpy="0 0 0"/>-->
+<!--    <parent link="mid_mount"/>-->
+<!--    <child link="kinect_link" />-->
+<!--  </joint>-->
 </robot>

Commit message: add realsense simulation

File: betago_description/urdf/betago/ridgeback_urdf_extras.xacro (robot description, xacro)
@@ -3,3 +3,6 @@
     <xacro:include filename="$(find betago_description)/urdf/betago/ridgeback_dual_ur5_description.urdf.xacro" />
 <!--    <xacro:include filename="$(find betago_description)/urdf/allegro_hand/dual_allegro_hand.xacro" />-->
+<!--    hand camera-->
+    <xacro:include filename="$(find betago_description)/urdf/sensors/kinect_prefix.urdf.xacro" />
+    <prefix_sensor_kinect prefix="left_hand" parent="left_ur_arm_ee_link" cam_px="0.05" cam_py="0" cam_pz="-0.1" cam_or="${pi}" cam_op="0" cam_oy="0"/>
 </robot>

File: betago_description/urdf/ridgeback/ridgeback.urdf.xacro (robot description, xacro)
@@ -279,7 +279,10 @@
   <!-- sensors -->
   <xacro:include filename="$(find betago_description)/urdf/sensors/kinect.urdf.xacro" />
-  <xacro:include filename="$(find betago_description)/urdf/sensors/kinect_prefix.urdf.xacro" />
   <sensor_kinect  parent="base_link"/>
-  <prefix_sensor_kinect prefix="left_hand" parent="left_ur_arm_ee_link" cam_px="0.05" cam_py="0" cam_pz="-0.1" cam_or="${pi}" cam_op="0" cam_oy="0"/>
+  <xacro:include filename="$(find realsense_gazebo_description)/urdf/_d435i.urdf.xacro"/>
+  <xacro:sensor_d435i parent="base_link" name="D435i_camera" topics_ns="D435i_camera"
+                      enable_pointCloud="true" unite_imu_method="linear_interpolation"> <!-- unite_imu_method can be false, copy or linear_interpolation -->
+    <origin xyz="0.25 0.0 0.7" rpy="0.0 0.0 0.0"/>
+  </xacro:sensor_d435i>
 <!--  <xacro:include filename="$(find betago_description)/urdf/sensors/kinect_gazebo.xacro" />-->
 <!--  <xacro:kinect_camera prefix="kinect" />-->

File: betago_description/urdf/sensors/kinect_prefix.urdf.xacro (robot description, xacro)
@@ -3,5 +3,5 @@
   <xacro:include filename="$(find betago_description)/urdf/sensors/kinect_gazebo_prefix.urdf.xacro"/>
 <!--  <xacro:include filename="$(find betago_description)/urdf/sensors/kinect_properties.urdf.xacro"/>-->
-<!--  <xacro:property name="kinect_cam_py" value="-0.0125"/>-->
+  <xacro:property name="kinect_cam_py" value="-0.0125"/>
   <!-- Parameterised in part by the values in kinect_properties.urdf.xacro -->
   <xacro:macro name="prefix_sensor_kinect" params="prefix parent cam_px cam_py cam_pz cam_or cam_op cam_oy">

Commit message: set mulitiple config for betago

File: betago_description/urdf/betago/ridgeback_urdf_extras.xacro (robot description, xacro)
@@ -5,4 +5,6 @@
 <!--    hand camera-->
     <xacro:include filename="$(find betago_description)/urdf/sensors/kinect_prefix.urdf.xacro" />
-    <prefix_sensor_kinect prefix="left_hand" parent="left_ur_arm_ee_link" cam_px="0.05" cam_py="0" cam_pz="-0.1" cam_or="${pi}" cam_op="0" cam_oy="0"/>
+    <xacro:if value="$(optenv BETAGO_ARM_KINECT 0)">
+        <prefix_sensor_kinect prefix="left_hand" parent="left_ur_arm_ee_link" cam_px="0.05" cam_py="0" cam_pz="-0.1" cam_or="${pi}" cam_op="0" cam_oy="0"/>
+    </xacro:if>
 </robot>

File: betago_description/urdf/ridgeback/ridgeback.urdf.xacro (robot description, xacro)
@@ -279,10 +279,14 @@
   <!-- sensors -->
   <xacro:include filename="$(find betago_description)/urdf/sensors/kinect.urdf.xacro" />
-  <sensor_kinect  parent="base_link"/>
+  <xacro:if value="$(optenv BETAGO_HEAD_KINECT 0)">
+    <xacro:sensor_kinect  parent="base_link"/>
+  </xacro:if>
   <xacro:include filename="$(find realsense_gazebo_description)/urdf/_d435i.urdf.xacro"/>
-  <xacro:sensor_d435i parent="base_link" name="D435i_camera" topics_ns="D435i_camera"
-                      enable_pointCloud="true" unite_imu_method="linear_interpolation"> <!-- unite_imu_method can be false, copy or linear_interpolation -->
-    <origin xyz="0.25 0.0 0.7" rpy="0.0 0.0 0.0"/>
-  </xacro:sensor_d435i>
+  <xacro:if value="$(optenv BETAGO_HEAD_D435i 0)">
+    <xacro:sensor_d435i parent="base_link" name="D435i_camera" topics_ns="D435i_camera"
+                        enable_pointCloud="true" unite_imu_method="linear_interpolation"> <!-- unite_imu_method can be false, copy or linear_interpolation -->
+      <origin xyz="0.25 0.0 0.7" rpy="0.0 0.0 0.0"/>
+    </xacro:sensor_d435i>
+  </xacro:if>
 <!--  <xacro:include filename="$(find betago_description)/urdf/sensors/kinect_gazebo.xacro" />-->
 <!--  <xacro:kinect_camera prefix="kinect" />-->

File: realsense/realsense_gazebo_description/urdf/_d435i.gazebo.xacro (robot description, xacro)
@@ -28,8 +28,8 @@
       <sensor name="${camera_name}color" type="camera">
         <camera name="${camera_name}">
-          <horizontal_fov>${69.4*deg_to_rad}</horizontal_fov>
+          <horizontal_fov>${90*deg_to_rad}</horizontal_fov>
           <image>
-            <width>1920</width>
-            <height>1080</height>
+            <width>640</width>
+            <height>480</height>
             <format>RGB_INT8</format>
           </image>
@@ -50,8 +50,8 @@
       <sensor name="${camera_name}ired1" type="camera">
         <camera name="${camera_name}">
-          <horizontal_fov>${85.2*deg_to_rad}</horizontal_fov>
+          <horizontal_fov>${86*deg_to_rad}</horizontal_fov>
           <image>
-            <width>1280</width>
-            <height>720</height>
+            <width>640</width>
+            <height>480</height>
             <format>L_INT8</format>
           </image>
@@ -74,6 +74,6 @@
           <horizontal_fov>${85.2*deg_to_rad}</horizontal_fov>
           <image>
-            <width>1280</width>
-            <height>720</height>
+            <width>640</width>
+            <height>480</height>
             <format>L_INT8</format>
           </image>
@@ -96,6 +96,6 @@
           <horizontal_fov>${85.2*deg_to_rad}</horizontal_fov>
           <image>
-            <width>1280</width>
-            <height>720</height>
+            <width>640</width>
+            <height>480</height>
           </image>
           <clip>
@@ -168,7 +168,7 @@
       <plugin name="${topics_ns}" filename="librealsense_gazebo_plugin.so">
         <prefix>${camera_name}</prefix>
-      	<depthUpdateRate>60.0</depthUpdateRate>
-      	<colorUpdateRate>60.0</colorUpdateRate>
-      	<infraredUpdateRate>60.0</infraredUpdateRate>
+      	<depthUpdateRate>30.0</depthUpdateRate>
+      	<colorUpdateRate>30.0</colorUpdateRate>
+      	<infraredUpdateRate>30.0</infraredUpdateRate>
       	<depthTopicName>depth/image_raw</depthTopicName>
       	<depthCameraInfoTopicName>depth/camera_info</depthCameraInfoTopicName>
