Commit message: set mulitiple config for betago

File: betago_description/urdf/ridgeback/ridgeback.urdf.xacro (robot description, xacro)
@@ -279,10 +279,14 @@
   <!-- sensors -->
   <xacro:include filename="$(find betago_description)/urdf/sensors/kinect.urdf.xacro" />
-  <sensor_kinect  parent="base_link"/>
+  <xacro:if value="$(optenv BETAGO_HEAD_KINECT 0)">
+    <xacro:sensor_kinect  parent="base_link"/>
+  </xacro:if>
   <xacro:include filename="$(find realsense_gazebo_description)/urdf/_d435i.urdf.xacro"/>
-  <xacro:sensor_d435i parent="base_link" name="D435i_camera" topics_ns="D435i_camera"
-                      enable_pointCloud="true" unite_imu_method="linear_interpolation"> <!-- unite_imu_method can be false, copy or linear_interpolation -->
-    <origin xyz="0.25 0.0 0.7" rpy="0.0 0.0 0.0"/>
-  </xacro:sensor_d435i>
+  <xacro:if value="$(optenv BETAGO_HEAD_D435i 0)">
+    <xacro:sensor_d435i parent="base_link" name="D435i_camera" topics_ns="D435i_camera"
+                        enable_pointCloud="false" unite_imu_method="linear_interpolation"> <!-- unite_imu_method can be false, copy or linear_interpolation -->
+      <origin xyz="0.25 0.0 0.7" rpy="0.0 0.0 0.0"/>
+    </xacro:sensor_d435i>
+  </xacro:if>
 <!--  <xacro:include filename="$(find betago_description)/urdf/sensors/kinect_gazebo.xacro" />-->
 <!--  <xacro:kinect_camera prefix="kinect" />-->

File: realsense/realsense_gazebo_description/urdf/_d435i.gazebo.xacro (robot description, xacro)
@@ -28,8 +28,8 @@
       <sensor name="${camera_name}color" type="camera">
         <camera name="${camera_name}">
-          <horizontal_fov>${69.4*deg_to_rad}</horizontal_fov>
+          <horizontal_fov>${90*deg_to_rad}</horizontal_fov>
           <image>
-            <width>1920</width>
-            <height>1080</height>
+            <width>640</width>
+            <height>480</height>
             <format>RGB_INT8</format>
           </image>
@@ -38,9 +38,9 @@
             <far>100</far>
           </clip>
-          <noise>
-            <type>gaussian</type>
-            <mean>0.0</mean>
-            <stddev>0.007</stddev>
-          </noise>
+<!--          <noise>-->
+<!--            <type>gaussian</type>-->
+<!--            <mean>0.0</mean>-->
+<!--            <stddev>0.007</stddev>-->
+<!--          </noise>-->
         </camera>
         <always_on>1</always_on>
@@ -50,8 +50,8 @@
       <sensor name="${camera_name}ired1" type="camera">
         <camera name="${camera_name}">
-          <horizontal_fov>${85.2*deg_to_rad}</horizontal_fov>
+          <horizontal_fov>${86*deg_to_rad}</horizontal_fov>
           <image>
-            <width>1280</width>
-            <height>720</height>
+            <width>640</width>
+            <height>480</height>
             <format>L_INT8</format>
           </image>
@@ -60,9 +60,9 @@
             <far>100</far>
           </clip>
-          <noise>
-            <type>gaussian</type>
-            <mean>0.0</mean>
-            <stddev>0.05</stddev>
-          </noise>
+<!--          <noise>-->
+<!--            <type>gaussian</type>-->
+<!--            <mean>0.0</mean>-->
+<!--            <stddev>0.05</stddev>-->
+<!--          </noise>-->
         </camera>
         <always_on>1</always_on>
@@ -74,6 +74,6 @@
           <horizontal_fov>${85.2*deg_to_rad}</horizontal_fov>
           <image>
-            <width>1280</width>
-            <height>720</height>
+            <width>640</width>
+            <height>480</height>
             <format>L_INT8</format>
           </image>
@@ -82,9 +82,9 @@
             <far>100</far>
           </clip>
-          <noise>
-            <type>gaussian</type>
-            <mean>0.0</mean>
-            <stddev>0.05</stddev>
-          </noise>
+<!--          <noise>-->
+<!--            <type>gaussian</type>-->
+<!--            <mean>0.0</mean>-->
+<!--            <stddev>0.05</stddev>-->
+<!--          </noise>-->
         </camera>
         <always_on>1</always_on>
@@ -96,6 +96,6 @@
           <horizontal_fov>${85.2*deg_to_rad}</horizontal_fov>
           <image>
-            <width>1280</width>
-            <height>720</height>
+            <width>640</width>
+            <height>480</height>
           </image>
           <clip>
@@ -103,9 +103,9 @@
             <far>100</far>
           </clip>
-          <noise>
-            <type>gaussian</type>
-            <mean>0.0</mean>
-            <stddev>0.100</stddev>
-          </noise>
+<!--          <noise>-->
+<!--            <type>gaussian</type>-->
+<!--            <mean>0.0</mean>-->
+<!--            <stddev>0.100</stddev>-->
+<!--          </noise>-->
         </camera>
         <always_on>1</always_on>
@@ -168,7 +168,7 @@
       <plugin name="${topics_ns}" filename="librealsense_gazebo_plugin.so">
         <prefix>${camera_name}</prefix>
-      	<depthUpdateRate>60.0</depthUpdateRate>
-      	<colorUpdateRate>60.0</colorUpdateRate>
-      	<infraredUpdateRate>60.0</infraredUpdateRate>
+      	<depthUpdateRate>30.0</depthUpdateRate>
+      	<colorUpdateRate>30.0</colorUpdateRate>
+      	<infraredUpdateRate>30.0</infraredUpdateRate>
       	<depthTopicName>depth/image_raw</depthTopicName>
       	<depthCameraInfoTopicName>depth/camera_info</depthCameraInfoTopicName>

Commit message: kinect navigation

File: betago_description/urdf/ridgeback/ridgeback.urdf.xacro (robot description, xacro)
@@ -283,8 +283,14 @@
   </xacro:if>
   <xacro:include filename="$(find realsense_gazebo_description)/urdf/_d435i.urdf.xacro"/>
+  <xacro:include filename="$(find realsense_gazebo_description)/urdf/_d435.urdf.xacro"/>
   <xacro:if value="$(optenv BETAGO_HEAD_D435i 0)">
     <xacro:sensor_d435i parent="base_link" name="D435i_camera" topics_ns="D435i_camera" enable_pointCloud="false" unite_imu_method="linear_interpolation"> <!-- unite_imu_method can be false, copy or linear_interpolation -->
       <origin xyz="0.25 0.0 0.7" rpy="0.0 0.0 0.0"/>
     </xacro:sensor_d435i>
+  </xacro:if>
+  <xacro:if value="$(optenv BETAGO_HEAD_D435 0)">
+    <xacro:sensor_d435 parent="base_link" name="D435_camera" topics_ns="D435_camera">
+      <origin xyz="0.25 0.0 0.7" rpy="0.0 0.0 0.0"/>
+    </xacro:sensor_d435>
   </xacro:if>
 <!--  <xacro:include filename="$(find betago_description)/urdf/sensors/kinect_gazebo.xacro" />-->
